File: UDB.kicad_sch (KiCad schematic)
At the start: 14 parts, among them J1 TYPE-C-31-M12_13, J2 X1224WRS-04-LPV01, U1 TPD4E05U06DQAR

Commit message: New version files and pertaining prod files added
Parts:
- removed L1: 60R@100MHz, Inductor_SMD:L_1206_3216Metric, symbol Unified-Daughterboard-rescue:L_Core_Ferrite-Device
- J2: value X1224WRS-04-LPV01 -> SM04B-SRSS-TB(LF)(SN); footprint locallib:PicoEZMate-Reinforced-Alt -> acheron_Connectors:SM04B-SRSS-TB(LF)(SN)_mounting-reliefs; LCSC Part Number C528030 -> C160404; Manufacturer XKB Connectivity -> JST; Manufacturer Part Number X1224WRS-04-LPV01 -> SM04B-SRSS-TB(LF)(SN)
Connections:
- net GNDPWR is gone; now on net GND: J1.S (SHIELD), MH2.1 (Pin_1)
